Commit message: add worlds/

File: urdf/legged_robot.urdf.xacro (robot description, xacro)
@@ -23,8 +23,8 @@
 izz="${m*(x*x+z*z)/12.}" />
 </macro>
-<!--link name="base_footprint"/>
+<link name="base_footprint"/>
 <gazebo reference="base_footprint">
 <turnGravityOff>false</turnGravityOff>
-</gazebo-->
+</gazebo>
   <!--body-->
   <link name="torso">
@@ -48,9 +48,9 @@
     </collision>
   </link>
-<!--joint name="base_link_joint" type="fixed">
+<joint name="base_link_joint" type="fixed">
 <origin xyz="0 0 0" rpy="0 0 0" />
 <parent link="base_footprint"/>
 <child link="torso" />
-</joint-->
+</joint>
 <!--legs macro-->
 <leg fr="fore" lr="left" transX="1" transY="1"/>
