Commit message: a little fix

File: urdf/leg.urdf.xacro (robot description, xacro)
@@ -1,4 +1,4 @@
 <?xml version="1.0"?>
-<robot name="wheel" xmlns:xacro="http://ros.org/wiki/xacro">
+<robot name="leg" xmlns:xacro="http://ros.org/wiki/xacro">
 <!-- legs -->
 <property name="leg_base_height" value="0.050" />
@@ -26,9 +26,9 @@
 <!--fr : front, rear ; lr: left, right -->
 <link name='base_${lr}_${fr}'>
-  <visual name='visual'>
+  <visual>
     <geometry>
       <cylinder length="${leg_base_height}" radius="${leg_base_radius}"/>
     </geometry>
-  <material name="White" />
+  <material name="Gray" />
    </visual>
   </link>
@@ -39,5 +39,5 @@
       <cylinder_inertia  m="${lower_leg_mass}" r="${lower_leg_radius}" h="${lower_leg_height}" />
     </inertial>
-    <collision name='collision'>
+    <collision>
       <origin xyz="0 0 ${lower_leg_height/2}" rpy="0 0 0" />
       <geometry>
@@ -45,10 +45,10 @@
       </geometry>
     </collision>
-    <visual name='visual'>
+    <visual>
       <origin xyz="0 0 ${lower_leg_height/2}" rpy="0 0 0" />
       <geometry>
 	<cylinder length="${lower_leg_height}" radius="${lower_leg_radius}"/>
       </geometry>
-    <material name="White" />
+    <material name="Gray" />
    </visual>
   </link>
@@ -59,5 +59,5 @@
       <cylinder_inertia  m="${upper_leg_mass}" r="${upper_leg_radius}" h="${upper_leg_height}" />
     </inertial>
-    <collision name='collision'>
+    <collision>
       <origin xyz="0 0 ${upper_leg_height/2}" rpy="0 0 0" />
       <geometry>
@@ -65,10 +65,10 @@
       </geometry>
     </collision>
-    <visual name='visual'>
+    <visual>
       <origin xyz="0 0 ${upper_leg_height/2}" rpy="0 0 0" />
       <geometry>
 	<cylinder length="${upper_leg_height}" radius="${upper_leg_radius}"/>
       </geometry>
-    <material name="White" />
+    <material name="Gray" />
    </visual>
   </link>
@@ -79,5 +79,5 @@
     <child link="base_${lr}_${fr}"/>
     <origin xyz="${transX*0.23} ${transY*0.17} 0.0" rpy="1.5707 0 0" />
-    <axis xyz="0 0 1" rpy="0 0 0"/>
+    <axis xyz="0 0 1"/>
     <limit effort="${limit_effort}" velocity="${limit_velocity}" lower="${limit_lower_1}" upper="${limit_upper_1}" />
   </joint>
@@ -87,5 +87,5 @@
     <child link="link_${lr}_${fr}_upper"/>
     <origin xyz="0 0 0" rpy="1.5707 0 0" />
-    <axis xyz="1 0 0" rpy="0 0 0"/>
+    <axis xyz="1 0 0"/>
     <limit effort="${limit_effort}" velocity="${limit_velocity}" lower="${limit_lower_2}" upper="${limit_upper_2}" />
   </joint>
@@ -94,9 +94,14 @@
     <parent link="link_${lr}_${fr}_upper"/>
     <child link="link_${lr}_${fr}_lower"/>
-    <origin xyz="0 0 0.30" rpy="0 0 0" />
-    <axis xyz="0 1 0" rpy="0 0 0"/>
+    <origin xyz="0 0 0.32" rpy="0 0 0" />
+    <axis xyz="0 1 0"/>
     <limit effort="${limit_effort}" velocity="${limit_velocity}" lower="${limit_lower_3}" upper="${limit_upper_3}" />
   </joint>
 <!-- =========gazebo reference============ -->
+<gazebo reference="base_${lr}_${fr}">
+<selfCollide value="false"/>
+<material>Gazebo/Gray</material>
+<turnGravityOff>true</turnGravityOff>
+</gazebo>
 <gazebo reference="link_${lr}_${fr}_lower">
 <selfCollide value="false"/>
@@ -106,5 +111,5 @@
 <kd  value="1.0" />
 <fdir1 value="1 0 0"/>
-<material>Gazebo/White</material>
+<material>Gazebo/Gray</material>
 <turnGravityOff>false</turnGravityOff>
 </gazebo>
@@ -116,5 +121,5 @@
 <kd  value="1.0" />
 <fdir1 value="1 0 0"/>
-<material>Gazebo/White</material>
+<material>Gazebo/Gray</material>
 <turnGravityOff>false</turnGravityOff>
 </gazebo>
@@ -122,5 +127,5 @@
 <transmission name="hinge_${lr}_${fr}_1_trans">
 <type>transmission_interface/SimpleTransmission</type>
-<joint name="hinge_${lr}_${fr}1">
+<joint name="hinge_${lr}_${fr}_1">
 <hardwareInterface>hardware_interface/EffortJointInterface</hardwareInterface>
 </joint>

File: urdf/legged_robot.urdf.xacro (robot description, xacro)
@@ -27,13 +27,8 @@
 <turnGravityOff>false</turnGravityOff>
 </gazebo>
-<joint name="base_link_joint" type="fixed">
-<origin xyz="0 0 0" rpy="0 0 0" />
-<parent link="base_footprint"/>
-<child link="torso" />
-</joint>
   <!--body-->
   <link name="torso">
     <inertial>
-    <origin xyz="0 0 0" rpy="0 0 0" />
+    <origin xyz="0 0 0"/>
     <mass value="${base_mass}" />
     <box_inertia  m="${base_mass}" x="${base_x_size}" y="${base_y_size}" z="${base_z_size}"/>
@@ -50,14 +45,24 @@
 	<box size="${base_x_size} ${base_y_size} ${base_z_size}"/>
       </geometry>
-    <material name="White" />
+    <material name="Gray" />
    </visual>
   </link>
-  <!--legs macro-->
-  <leg fr="fore" lr="left" transX="1" transY="1"/>
-  <leg fr="fore" lr="right" transX="1" transY="-1"/>
-  <leg fr="rear" lr="left" transX="-1" transY="1"/>
-  <leg fr="rear" lr="right" transX="-1" transY="-1"/>
+<joint name="base_link_joint" type="fixed">
+<origin xyz="0 0 0" rpy="0 0 0" />
+<parent link="base_footprint"/>
+<child link="torso" />
+</joint>
+<!--legs macro-->
+<leg fr="fore" lr="left" transX="1" transY="1"/>
+<leg fr="fore" lr="right" transX="1" transY="-1"/>
+<leg fr="rear" lr="left" transX="-1" transY="1"/>
+<leg fr="rear" lr="right" transX="-1" transY="-1"/>
+  <!-- =========gazebo reference============ -->
+<gazebo reference="torso">
+<material>Gazebo/Black</material>
+<turnGravityOff>false</turnGravityOff>
+</gazebo>
   <!--gazebo>
-  <plugin name="gazebo_legged_robot_plugin" filename="libgazebo_legged_robot_plugin.so" >
+  <plugin name="gazebo_legged_robot_walking_plugin" filename="libgazebo_legged_robot_walking_plugin.so" >
     <hinge_lf1>hinge_left_fore_1</hinge_lf1>
     <hinge_lf2>hinge_left_fore_2</hinge_lf2>

Commit message: fix gazebo bug to add collision and inertial tags into only visual tag link.

File: urdf/leg.urdf.xacro (robot description, xacro)
@@ -4,4 +4,5 @@
 <property name="leg_base_height" value="0.050" />
 <property name="leg_base_radius" value="0.025" />
+<property name="leg_base_mass" value="0.5" />
 <property name="lower_leg_height" value="0.3" />
 <property name="lower_leg_radius" value="0.02" />
@@ -32,8 +33,19 @@
   <material name="Gray" />
    </visual>
+   <collision>
+   <origin xyz="0 0 0" rpy="0 0 0 " />
+	<geometry>
+	<cylinder length="${leg_base_height}" radius="${leg_base_radius}"/>
+	</geometry>
+</collision>
+<inertial>
+     <origin xyz="0 0 0" />
+      <mass value="${leg_base_mass}" />
+      <cylinder_inertia  m="${leg_base_mass}" r="${leg_base_radius}" h="${leg_base_height}" />
+    </inertial>
   </link>
 <link name='link_${lr}_${fr}_lower'>
     <inertial>
-     <origin xyz="0 0 ${lower_leg_height/2}" rpy="0 0 0" />
+     <origin xyz="0 0 ${lower_leg_height/2}"/>
       <mass value="${lower_leg_mass}" />
       <cylinder_inertia  m="${lower_leg_mass}" r="${lower_leg_radius}" h="${lower_leg_height}" />
@@ -55,5 +67,5 @@
   <link name='link_${lr}_${fr}_upper'>
     <inertial>
-      <origin xyz="0 0 ${upper_leg_height/2}" rpy="0 0 0" />
+      <origin xyz="0 0 ${upper_leg_height/2}"/>
       <mass value="${upper_leg_mass}" />
       <cylinder_inertia  m="${upper_leg_mass}" r="${upper_leg_radius}" h="${upper_leg_height}" />
@@ -94,5 +106,5 @@
     <parent link="link_${lr}_${fr}_upper"/>
     <child link="link_${lr}_${fr}_lower"/>
-    <origin xyz="0 0 0.32" rpy="0 0 0" />
+    <origin xyz="0 0 0.30" rpy="0 0 0" />
     <axis xyz="0 1 0"/>
     <limit effort="${limit_effort}" velocity="${limit_velocity}" lower="${limit_lower_3}" upper="${limit_upper_3}" />

File: urdf/legged_robot.urdf.xacro (robot description, xacro)
@@ -1,4 +1,4 @@
 <?xml version='1.0'?>
-<robot name="legged_robot" xmlns:xacro="http://www.ros.org/wiki/xacro">
+<robot name="legged_robot" xmlns:xacro="http://ros.org/wiki/xacro">
 <!-- Included URDF/XACRO Files -->
 <xacro:include filename="$(find legged_robot)/urdf/materials.urdf.xacro" />
@@ -23,8 +23,8 @@
 izz="${m*(x*x+z*z)/12.}" />
 </macro>
-<link name="base_footprint"/>
+<!--link name="base_footprint"/>
 <gazebo reference="base_footprint">
 <turnGravityOff>false</turnGravityOff>
-</gazebo>
+</gazebo-->
   <!--body-->
   <link name="torso">
@@ -34,11 +34,5 @@
     <box_inertia  m="${base_mass}" x="${base_x_size}" y="${base_y_size}" z="${base_z_size}"/>
     </inertial>
-    <collision name='collision'>
-    <origin xyz="0 0 0" rpy="0 0 0" />
-      <geometry>
-	<box size="${base_x_size} ${base_y_size} ${base_z_size}"/>
-      </geometry>
-    </collision>
-    <visual name='visual'>
+    <visual>
     <origin xyz="0 0 0" rpy="0 0 0" />
       <geometry>
@@ -47,10 +41,16 @@
     <material name="Gray" />
    </visual>
+   <collision>
+    <origin xyz="0 0 0" rpy="0 0 0" />
+      <geometry>
+	<box size="${base_x_size} ${base_y_size} ${base_z_size}"/>
+      </geometry>
+    </collision>
   </link>
-<joint name="base_link_joint" type="fixed">
+<!--joint name="base_link_joint" type="fixed">
 <origin xyz="0 0 0" rpy="0 0 0" />
 <parent link="base_footprint"/>
 <child link="torso" />
-</joint>
+</joint-->
 <!--legs macro-->
 <leg fr="fore" lr="left" transX="1" transY="1"/>
@@ -60,5 +60,5 @@
   <!-- =========gazebo reference============ -->
 <gazebo reference="torso">
-<material>Gazebo/Black</material>
+<material>Gazebo/Gray</material>
 <turnGravityOff>false</turnGravityOff>
 </gazebo>

Commit message: add trot control(incomplete)

File: urdf/leg.urdf.xacro (robot description, xacro)
@@ -6,21 +6,28 @@
 <property name="leg_base_mass" value="0.5" />
 <property name="lower_leg_height" value="0.3" />
-<property name="lower_leg_radius" value="0.02" />
+<property name="lower_leg_radius" value="0.01" />
 <property name="lower_leg_mass" value="2.0" />
-<property name="upper_leg_height" value="0.3" />
+<property name="upper_leg_height" value="0.20" />
 <property name="upper_leg_radius" value="0.02" />
 <property name="upper_leg_mass" value="2.0" />
-<property name="limit_effort" value="30" />
-<property name="limit_velocity" value="1.0" />
-<property name="limit_lower_1" value="-1.57" />
-<property name="limit_upper_1" value="1.57" />
+<property name="limit_effort" value="1000" />
+<property name="limit_velocity" value="100.0" />
+<property name="limit_lower_1" value="-0.3926875" />
+<property name="limit_upper_1" value="0.785" />
 <property name="limit_lower_2" value="-0.1963" />
 <property name="limit_upper_2" value="0.1963" />
-<property name="limit_lower_3" value="-1.57" />
-<property name="limit_upper_3" value="0" />
+<property name="limit_lower_3" value="-0.785" />
+<property name="limit_upper_3" value="0.785" />
+<property name="sphere_r" value="0.02" />
+<property name="sphere_mass" value="0.02" />
 <macro name="cylinder_inertia" params="m r h">
 <inertia  ixx="${m*(3*r*r+h*h)/12}" ixy = "0" ixz = "0"
 iyy="${m*(3*r*r+h*h)/12}" iyz = "0"
 izz="${m*r*r/2}" />
+</macro>
+<macro name="sphere_inertia" params="m r">
+<inertia  ixx="${m*(2*r*r)/5}" ixy = "0" ixz = "0"
+iyy="${m*(2*r*r)/5}}" iyz = "0"
+izz="${m*(2*r*r)/5}" />
 </macro>
 <xacro:macro name="leg" params="fr lr transX transY">
@@ -31,5 +38,5 @@
       <cylinder length="${leg_base_height}" radius="${leg_base_radius}"/>
     </geometry>
-  <material name="Gray" />
+  <material name="Black" />
    </visual>
    <collision>
@@ -45,4 +52,28 @@
     </inertial>
   </link>
+<link name='serbo_${lr}_${fr}'>
+  <visual>
+    <geometry>
+      <cylinder length="${leg_base_height}" radius="${leg_base_radius}"/>
+    </geometry>
+  <material name="Black" />
+   </visual>
+   <collision>
+   <origin xyz="0 0 0" rpy="0 0 0 " />
+	<geometry>
+	<cylinder length="${leg_base_height}" radius="${leg_base_radius}"/>
+	</geometry>
+</collision>
+<inertial>
+     <origin xyz="0 0 0" />
+      <mass value="${leg_base_mass}" />
+      <cylinder_inertia  m="${leg_base_mass}" r="${leg_base_radius}" h="${leg_base_height}" />
+    </inertial>
+  </link>
+   <joint name="serbo_${lr}_${fr}_joint" type="fixed">
+    <parent link="link_${lr}_${fr}_upper"/>
+    <child  link="serbo_${lr}_${fr}"/>
+    <origin xyz="0 0 ${upper_leg_height}" rpy="1.5707 0 0"/>
+  </joint>
 <link name='link_${lr}_${fr}_lower'>
     <inertial>
@@ -85,10 +116,34 @@
    </visual>
   </link>
+  <link name='ball_${lr}_${fr}'>
+  <visual>
+    <geometry>
+      <sphere radius="${sphere_r}"/>
+    </geometry>
+  <material name="Black" />
+   </visual>
+   <collision>
+   <origin xyz="0 0 0" rpy="0 0 0 " />
+	<geometry>
+	<sphere radius="${sphere_r}"/>
+	</geometry>
+</collision>
+<inertial>
+     <origin xyz="0 0 0" />
+      <mass value="${sphere_mass}" />
+      <sphere_inertia  m="${sphere_mass}" r="${sphere_r}" />
+    </inertial>
+  </link>
+  <joint name="ball_${lr}_${fr}_joint" type="fixed">
+    <parent link="link_${lr}_${fr}_lower"/>
+    <child  link="ball_${lr}_${fr}"/>
+    <origin xyz="0 0 ${lower_leg_height}" rpy="0 0 0"/>
+  </joint>
   <!--joint-->
   <!--1st joint-->
   <joint type="revolute" name="hinge_${lr}_${fr}_1">
-    <parent link="torso"/>
+    <parent link="base_link"/>
     <child link="base_${lr}_${fr}"/>
-    <origin xyz="${transX*0.23} ${transY*0.17} 0.0" rpy="1.5707 0 0" />
+    <origin xyz="${transX*0.23} ${transY*0.17} 0.0" rpy="1.5707 0.785 0" />
     <axis xyz="0 0 1"/>
     <limit effort="${limit_effort}" velocity="${limit_velocity}" lower="${limit_lower_1}" upper="${limit_upper_1}" />
@@ -104,8 +159,8 @@
   <!--3rd joint-->
   <joint type="revolute" name="hinge_${lr}_${fr}_3">
-    <parent link="link_${lr}_${fr}_upper"/>
+    <parent link="serbo_${lr}_${fr}"/>
     <child link="link_${lr}_${fr}_lower"/>
-    <origin xyz="0 0 0.30" rpy="0 0 0" />
-    <axis xyz="0 1 0"/>
+    <origin xyz="0 0 0" rpy="0 1.5707 0" />
+    <axis xyz="1 0 0"/>
     <limit effort="${limit_effort}" velocity="${limit_velocity}" lower="${limit_lower_3}" upper="${limit_upper_3}" />
   </joint>
@@ -113,11 +168,21 @@
 <gazebo reference="base_${lr}_${fr}">
 <selfCollide value="false"/>
+<material>Gazebo/Black</material>
+<turnGravityOff>false</turnGravityOff>
+</gazebo>
+<gazebo reference="link_${lr}_${fr}_lower">
+<selfCollide value="false"/>
+<mu1 value="10000.0"/>
+<mu2 value="10000.0"/>
+<kp  value="10000000.0" />
+<kd  value="1.0" />
+<fdir1 value="1 0 0"/>
 <material>Gazebo/Gray</material>
-<turnGravityOff>true</turnGravityOff>
-</gazebo>
-<gazebo reference="link_${lr}_${fr}_lower">
-<selfCollide value="false"/>
-<mu1 value="1.0"/>
-<mu2 value="1.0"/>
+<turnGravityOff>false</turnGravityOff>
+</gazebo>
+<gazebo reference="link_${lr}_${fr}_upper">
+<selfCollide value="false"/>
+<mu1 value="10000.0"/>
+<mu2 value="10000.0"/>
 <kp  value="10000000.0" />
 <kd  value="1.0" />
@@ -126,12 +191,22 @@
 <turnGravityOff>false</turnGravityOff>
 </gazebo>
-<gazebo reference="link_${lr}_${fr}_upper">
-<selfCollide value="false"/>
-<mu1 value="1.0"/>
-<mu2 value="1.0"/>
-<kp  value="10000000.0" />
-<kd  value="1.0" />
-<fdir1 value="1 0 0"/>
-<material>Gazebo/Gray</material>
+<gazebo reference="ball_${lr}_${fr}">
+<selfCollide value="false"/>
+<mu1 value="10000.0"/>
+<mu2 value="10000.0"/>
+<kp  value="10000000.0" />
+<kd  value="1.0" />
+<fdir1 value="1 0 0"/>
+<material>Gazebo/Black</material>
+<turnGravityOff>false</turnGravityOff>
+</gazebo>
+<gazebo reference="serbo_${lr}_${fr}">
+<selfCollide value="false"/>
+<mu1 value="10000.0"/>
+<mu2 value="10000.0"/>
+<kp  value="10000000.0" />
+<kd  value="1.0" />
+<fdir1 value="1 0 0"/>
+<material>Gazebo/Black</material>
 <turnGravityOff>false</turnGravityOff>
 </gazebo>

File: urdf/legged_robot.urdf.xacro (robot description, xacro)
@@ -5,16 +5,8 @@
 <xacro:include filename="$(find legged_robot)/urdf/leg.urdf.xacro" />
 <!--configuration-->
-<property name="base_mass" value="10.0" />
+<property name="base_mass" value="5.0" />
 <property name="base_x_size" value="0.5" />
 <property name="base_y_size" value="0.3" />
 <property name="base_z_size" value="0.05" />
-<property name="leg_base_height" value="0.050" />
-<property name="leg_base_radius" value="0.025" />
-<property name="lower_leg_height" value="0.3" />
-<property name="lower_leg_radius" value="0.02" />
-<property name="lower_leg_mass" value="2.0" />
-<property name="upper_leg_height" value="0.3" />
-<property name="upper_leg_radius" value="0.02" />
-<property name="upper_leg_mass" value="2.0" />
 <!--macro-->
 <macro name="box_inertia" params="m x y z">
@@ -28,5 +20,5 @@
 </gazebo>
   <!--body-->
-  <link name="torso">
+  <link name="base_link">
     <inertial>
     <origin xyz="0 0 0"/>
@@ -51,5 +43,5 @@
 <origin xyz="0 0 0" rpy="0 0 0" />
 <parent link="base_footprint"/>
-<child link="torso" />
+<child link="base_link" />
 </joint>
 <!--legs macro-->
@@ -59,5 +51,5 @@
 <leg fr="rear" lr="right" transX="-1" transY="-1"/>
   <!-- =========gazebo reference============ -->
-<gazebo reference="torso">
+<gazebo reference="base_link">
 <material>Gazebo/Gray</material>
 <turnGravityOff>false</turnGravityOff>
@@ -65,4 +57,5 @@
 <gazebo>
   <plugin name="gazebo_ros_legged_robot" filename="libgazebo_ros_legged_robot.so" >
+    <commandTopic>/legged_robot/cmd_ang</commandTopic>
     <hinge_lf1>hinge_left_front_1</hinge_lf1>
     <hinge_lf2>hinge_left_front_2</hinge_lf2>
